Commit message: Stable

File: clover_description/urdf/clover/clover4.xacro (robot description, xacro)
@@ -14,5 +14,5 @@
   <!-- Create camera plugin -->
   <xacro:if value="$(arg main_camera)">
-    <xacro:rpi_cam name="main_camera" parent="base_link" x="0.055" y="0.0" z="-0.03" roll="0" pitch="${pi/2}" yaw="0" width="320" height="240" rate="40" do_throttling="$(arg maintain_camera_rate)"/>
+    <xacro:rpi_cam name="main_camera" parent="base_link" x="0.055" y="0.0" z="-0.03" roll="0" pitch="${pi/2}" yaw="0" width="640" height="480" rate="40" do_throttling="$(arg maintain_camera_rate)"/>
   </xacro:if>
   <!-- Instantiate LED strip -->

File: clover_description/urdf/sensors/rpi_cam.urdf.xacro (robot description, xacro)
@@ -2,5 +2,5 @@
 <robot name="rpi_camera" xmlns:xacro="http://ros.org/wiki/xacro">
   <xacro:include filename="../camera_sensor.urdf.xacro"/>
-  <xacro:macro name="rpi_cam" params="name:=rpi_cam parent x:=0 y:=0 z:=0 roll:=0 pitch:=0 yaw:=0 width:=320 height:=240 rate:=40 do_throttling:=false">
+  <xacro:macro name="rpi_cam" params="name:=rpi_cam parent x:=0 y:=0 z:=0 roll:=0 pitch:=0 yaw:=0 width:=640 height:=480 rate:=40 do_throttling:=false">
     <joint name="${name}_joint" type="fixed">
       <origin xyz="${x} ${y} ${z}"
@@ -51,5 +51,5 @@
       height="${height}"
       rate="${rate}"
-      horizontal_fov="${120 * pi / 180}"
+      horizontal_fov="${90 * pi / 180}"
       do_throttling="${do_throttling}"
     />
